File: Solar Sensor PCB/SolarSensorATMEGA328_PCB.kicad_pcb (KiCad board)
At the start: 2 copper layers, 44.9 x 44.9 mm, 33 parts, among them P1 I2C, P10 I2C, P2 SERIAL, P3 ID, P4 ISP, P5 LOGO2, P6 PCB, P8 ADC, P9 PROG, SW1 SWA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

Commit message: large update of firmware & PCB changes
This version works
Parts:
- C10, C9: value 22pf -> 22p
- C5, C7, C8: value 100nf -> 100n
- C6: value 100uf -> 100u
- D1: footprint REInnovationFootprint:TH_LED-5MM_larg_pad -> REInnovationFootprint:LED-5MM_larg_pad
- moved D1 0.63 mm to (148.6, 111.1)
Connections:
- D1 pad 1: Net-(C1-Pad2) -> GND
- D1 pad 2: GND -> Net-(C1-Pad2)
- U1 pad 3: Net-(C1-Pad2) -> GND
- U1 pad 4: GND -> Net-(C1-Pad2)
Routing:
- net GND: track 223.5 -> 227.1 mm
- net Net-(C1-Pad2): track 14.4 -> 17.4 mm
Other:
- rule pad_to_mask_clearance: 0.1 -> 0
