File: Solar Sensor PCB/SolarSensorATMEGA328_PCB.sch (KiCad schematic (older format))
At the start: 5 parts, among them P1 I2C, P2 SERIAL, P5 LOGO2, P6 PCB, P7 ENC

Commit message: updated new PCB version
Parts:
- added C11: 100n, REInnovationFootprint:SM_C_0805, symbol device:C
- added J1: ANALOG, REInnovationFootprint:SIL-3_screw_terminal, symbol Connector_Generic:Conn_01x03
- added R2: 10k, REInnovationFootprint:SM0805, symbol device:R
- P6: footprint REInnovationFootprint:PCB_45_45_Cut_Out_Solar_Sensor -> REInnovationFootprint:PCB_SolarSensorATMEGA328_PCB_design_v2
Connections:
- net ATMega328/D6: now also R2.1
- net GND: now also C11.2, J1.3 (Pin_3)
- net VCC: now also J1.1 (Pin_1)
- new net IRR_A: C11.1, J1.2 (Pin_2), R2.2
Other:
- note added: "Analog"
- note added: "Low Pass Filter\nCut off 150 Hz"
- moved on the sheet: P2

Commit message: Updated firmware.
Sorted serial requests
Parts:
- C11: JLCPCB Add (none) -> Y; LCSC (none) -> C49678
- R2: JLCPCB Add (none) -> Y; LCSC (none) -> C17414
Changed lines of the file:
@@
 F 2 "REInnovationFootprint:SM0805" V 5430 3600 50  0001 C CNN
 F 3 "~" H 5500 3600 50  0001 C CNN
+F 4 "C17414" H 5500 3600 50  0001 C CNN "LCSC"
+F 5 "Y" H 5500 3600 50  0001 C CNN "JLCPCB Add"
 	1    5500 3600
 	0    1    1    0
@@
 F 2 "REInnovationFootprint:SM_C_0805" H 5188 3750 50  0001 C CNN
 F 3 "~" H 5150 3900 50  0001 C CNN
+F 4 "C49678" H 5150 3900 50  0001 C CNN "LCSC"
+F 5 "Y" H 5150 3900 50  0001 C CNN "JLCPCB Add"
 	1    5150 3900
 	1    0    0    -1
