File: Solar Sensor PCB/atmega328.sch (KiCad schematic (older format))
At the start: 19 parts, among them P10 I2C, P3 ID, P4 ISP, P9 PROG, SW1 SWA, SW2 RST, U4 ATmega328P-AU, Y1 8MHz_XTAL

Commit message: large update of firmware & PCB changes
This version works
Parts:
- C10, C9: value 22pf -> 22p; JLCPCB Add (none) -> Y; LCSC (none) -> C1804
- C5, C7, C8: value 100nf -> 100n; JLCPCB Add (none) -> Y; LCSC (none) -> C49678
- C6: value 100uf -> 100u; JLCPCB Add (none) -> Y; LCSC (none) -> C164071
Changed lines of the file:
@@
 P 7550 2800
 F 0 "C10" V 7700 2850 50  0000 C CNN
-F 1 "22pf" V 7700 2700 50  0000 C CNN
+F 1 "22p" V 7700 2700 50  0000 C CNN
 F 2 "REInnovationFootprint:SM_C_0805" H 7588 2650 50  0001 C CNN
 F 3 "~" H 7550 2800 50  0001 C CNN
+F 4 "C1804" H 7550 2800 50  0001 C CNN "LCSC"
+F 5 "Y" H 7550 2800 50  0001 C CNN "JLCPCB Add"
 	1    7550 2800
 	0    1    1    0
@@
 P 7550 2300
 F 0 "C9" V 7700 2350 50  0000 C CNN
-F 1 "22pf" V 7700 2200 50  0000 C CNN
+F 1 "22p" V 7700 2200 50  0000 C CNN
 F 2 "REInnovationFootprint:SM_C_0805" H 7588 2150 50  0001 C CNN
 F 3 "~" H 7550 2300 50  0001 C CNN
+F 4 "C1804" H 7550 2300 50  0001 C CNN "LCSC"
+F 5 "Y" H 7550 2300 50  0001 C CNN "JLCPCB Add"
 	1    7550 2300
 	0    1    1    0
@@
 P 7500 3700
 F 0 "C8" V 7650 3800 50  0000 C CNN
-F 1 "100nf" V 7350 3800 50  0000 C CNN
+F 1 "100n" V 7350 3800 50  0000 C CNN
 F 2 "REInnovationFootprint:SM_C_0805" H 7538 3550 50  0001 C CNN
 F 3 "~" H 7500 3700 50  0001 C CNN
+F 4 "C49678" H 7500 3700 50  0001 C CNN "LCSC"
+F 5 "Y" H 7500 3700 50  0001 C CNN "JLCPCB Add"
 	1    7500 3700
 	0    1    1    0
@@
 P 4600 3550
 F 0 "C7" H 4650 3450 50  0000 C CNN
-F 1 "100nf" V 4500 3750 50  0000 C CNN
+F 1 "100n" V 4500 3750 50  0000 C CNN
 F 2 "REInnovationFootprint:SM_C_0805" H 4638 3400 50  0001 C CNN
 F 3 "~" H 4600 3550 50  0001 C CNN
+F 4 "C49678" H 4600 3550 50  0001 C CNN "LCSC"
+F 5 "Y" H 4600 3550 50  0001 C CNN "JLCPCB Add"
 	1    4600 3550
 	-1   0    0    1
@@
 P 4300 3550
 F 0 "C6" H 4100 3650 50  0000 L CNN
-F 1 "100uf" V 4150 3350 50  0000 L CNN
+F 1 "100u" V 4150 3350 50  0000 L CNN
 F 2 "REInnovationFootprint:SM_6.3x7.7" H 4338 3400 50  0001 C CNN
 F 3 "~" H 4300 3550 50  0001 C CNN
+F 4 "C164071" H 4300 3550 50  0001 C CNN "LCSC"
+F 5 "Y" H 4300 3550 50  0001 C CNN "JLCPCB Add"
 	1    4300 3550
 	1    0    0    -1
@@
 P 4200 2050
 F 0 "C5" H 4250 1950 50  0000 C CNN
-F 1 "100nf" V 4100 2250 50  0000 C CNN
+F 1 "100n" V 4100 2250 50  0000 C CNN
 F 2 "REInnovationFootprint:SM_C_0805" H 4238 1900 50  0001 C CNN
 F 3 "~" H 4200 2050 50  0001 C CNN
+F 4 "C49678" H 4200 2050 50  0001 C CNN "LCSC"
+F 5 "Y" H 4200 2050 50  0001 C CNN "JLCPCB Add"
 	1    4200 2050
 	-1   0    0    1

Commit message: Updated PCB and Firmware
Added 3D models to new Kicad PCB
Connections:
- net A0: now also P3.5; no longer P3.1
- net A2: now also P3.1; no longer P3.5
Changed lines of the file:
@@
 Wire Wire Line
 	2600 4250 2450 4250
-Text Label 2450 4250 2    50   ~ 0
+Text Label 2450 4050 2    50   ~ 0
 A2
 Text Label 2450 4150 2    50   ~ 0
 A1
-Text Label 2450 4050 2    50   ~ 0
+Text Label 2450 4250 2    50   ~ 0
 A0
 Wire Wire Line

Commit message: Updated firmware.
Sorted serial requests
Parts:
- D2: value LED0 -> OUT
Changed lines of the file:
@@
 AR Path="/60FF06B8/60FFEEC0" Ref="D2"  Part="1"
 F 0 "D2" V 1900 3300 50  0000 R CNN
-F 1 "LED0" V 1550 3300 50  0000 R CNN
+F 1 "OUT" V 1550 3300 50  0000 R CNN
 F 2 "REInnovationFootprint:SM0805_LED" H 1800 3300 50  0001 C CNN
 F 3 "~" H 1800 3300 50  0001 C CNN
